File: ring.sch (EAGLE design)
At the start: 22 parts

Commit message: dimensions
Parts:
- R1, R10, R2, R3, R4, R5, R6, R7, R8, R9: value (none) -> 330R
Changed lines of the file:
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@@
 <?xml version="1.0" encoding="utf-8"?>
 <!DOCTYPE eagle SYSTEM "eagle.dtd">
-<eagle version="7.6.0">
+<eagle version="7.1.0">
 <drawing>
 <settings>
@@
 <part name="LED9" library="led" deviceset="LED" device="KA-3528ASYC"/>
 <part name="LED10" library="led" deviceset="LED" device="KA-3528ASYC"/>
-<part name="R1" library="rcl" deviceset="R-EU_" device="R0402"/>
-<part name="R2" library="rcl" deviceset="R-EU_" device="R0402"/>
-<part name="R3" library="rcl" deviceset="R-EU_" device="R0402"/>
-<part name="R4" library="rcl" deviceset="R-EU_" device="R0402"/>
-<part name="R5" library="rcl" deviceset="R-EU_" device="R0402"/>
-<part name="R6" library="rcl" deviceset="R-EU_" device="R0402"/>
-<part name="R7" library="rcl" deviceset="R-EU_" device="R0402"/>
-<part name="R8" library="rcl" deviceset="R-EU_" device="R0402"/>
-<part name="R9" library="rcl" deviceset="R-EU_" device="R0402"/>
-<part name="R10" library="rcl" deviceset="R-EU_" device="R0402"/>
+<part name="R1" library="rcl" deviceset="R-EU_" device="R0402" value="330R"/>
+<part name="R2" library="rcl" deviceset="R-EU_" device="R0402" value="330R"/>
+<part name="R3" library="rcl" deviceset="R-EU_" device="R0402" value="330R"/>
+<part name="R4" library="rcl" deviceset="R-EU_" device="R0402" value="330R"/>
+<part name="R5" library="rcl" deviceset="R-EU_" device="R0402" value="330R"/>
+<part name="R6" library="rcl" deviceset="R-EU_" device="R0402" value="330R"/>
+<part name="R7" library="rcl" deviceset="R-EU_" device="R0402" value="330R"/>
+<part name="R8" library="rcl" deviceset="R-EU_" device="R0402" value="330R"/>
+<part name="R9" library="rcl" deviceset="R-EU_" device="R0402" value="330R"/>
+<part name="R10" library="rcl" deviceset="R-EU_" device="R0402" value="330R"/>
 <part name="PAD1" library="wirepad" deviceset="SMD2" device=""/>
 <part name="PAD2" library="wirepad" deviceset="SMD2" device=""/>

Commit message: fin
Parts:
- R1, R10, R2, R3, R4, R5, R6, R7, R8, R9: device rcl:R-EU_R0402 -> rcl:R-EU_R0805W
Changed lines of the file:
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@@
 <layers>
 <layer number="1" name="Top" color="4" fill="1" visible="no" active="no"/>
+<layer number="2" name="Route2" color="1" fill="3" visible="no" active="no"/>
+<layer number="3" name="Route3" color="4" fill="3" visible="no" active="no"/>
+<layer number="4" name="Route4" color="1" fill="4" visible="no" active="no"/>
+<layer number="5" name="Route5" color="4" fill="4" visible="no" active="no"/>
+<layer number="6" name="Route6" color="1" fill="8" visible="no" active="no"/>
+<layer number="7" name="Route7" color="4" fill="8" visible="no" active="no"/>
+<layer number="8" name="Route8" color="1" fill="2" visible="no" active="no"/>
+<layer number="9" name="Route9" color="4" fill="2" visible="no" active="no"/>
+<layer number="10" name="Route10" color="1" fill="7" visible="no" active="no"/>
+<layer number="11" name="Route11" color="4" fill="7" visible="no" active="no"/>
+<layer number="12" name="Route12" color="1" fill="5" visible="no" active="no"/>
+<layer number="13" name="Route13" color="4" fill="5" visible="no" active="no"/>
+<layer number="14" name="Route14" color="1" fill="6" visible="no" active="no"/>
+<layer number="15" name="Route15" color="4" fill="6" visible="no" active="no"/>
 <layer number="16" name="Bottom" color="1" fill="1" visible="no" active="no"/>
 <layer number="17" name="Pads" color="2" fill="1" visible="no" active="no"/>
@@
 <part name="LED9" library="led" deviceset="LED" device="KA-3528ASYC"/>
 <part name="LED10" library="led" deviceset="LED" device="KA-3528ASYC"/>
-<part name="R1" library="rcl" deviceset="R-EU_" device="R0402" value="330R"/>
-<part name="R2" library="rcl" deviceset="R-EU_" device="R0402" value="330R"/>
-<part name="R3" library="rcl" deviceset="R-EU_" device="R0402" value="330R"/>
-<part name="R4" library="rcl" deviceset="R-EU_" device="R0402" value="330R"/>
-<part name="R5" library="rcl" deviceset="R-EU_" device="R0402" value="330R"/>
-<part name="R6" library="rcl" deviceset="R-EU_" device="R0402" value="330R"/>
-<part name="R7" library="rcl" deviceset="R-EU_" device="R0402" value="330R"/>
-<part name="R8" library="rcl" deviceset="R-EU_" device="R0402" value="330R"/>
-<part name="R9" library="rcl" deviceset="R-EU_" device="R0402" value="330R"/>
-<part name="R10" library="rcl" deviceset="R-EU_" device="R0402" value="330R"/>
+<part name="R1" library="rcl" deviceset="R-EU_" device="R0805W" value="330R"/>
+<part name="R2" library="rcl" deviceset="R-EU_" device="R0805W" value="330R"/>
+<part name="R3" library="rcl" deviceset="R-EU_" device="R0805W" value="330R"/>
+<part name="R4" library="rcl" deviceset="R-EU_" device="R0805W" value="330R"/>
+<part name="R5" library="rcl" deviceset="R-EU_" device="R0805W" value="330R"/>
+<part name="R6" library="rcl" deviceset="R-EU_" device="R0805W" value="330R"/>
+<part name="R7" library="rcl" deviceset="R-EU_" device="R0805W" value="330R"/>
+<part name="R8" library="rcl" deviceset="R-EU_" device="R0805W" value="330R"/>
+<part name="R9" library="rcl" deviceset="R-EU_" device="R0805W" value="330R"/>
+<part name="R10" library="rcl" deviceset="R-EU_" device="R0805W" value="330R"/>
 <part name="PAD1" library="wirepad" deviceset="SMD2" device=""/>
 <part name="PAD2" library="wirepad" deviceset="SMD2" device=""/>

Commit message: new
Parts:
- added LED11, LED12, LED13, LED14, LED15, LED16: (no value), led:LEDKA-3528ASYC
- added PAD3, PAD4: (no value), wirepad:SMD2
- added R11, R12, R13, R14, R15, R16: 330R, rcl:R-EU_R0805W
Connections:
- new net N$11: PAD3.P, R10.2, R11.2, R12.2, R13.2, R14.2, R15.2, R16.2, R9.2
- new net N$12: LED10.C, LED11.C, LED12.C, LED13.C, LED14.C, LED15.C, LED16.C, LED9.C, PAD4.P
- new net N$15: LED11.A, R11.1
- new net N$16: LED12.A, R12.1
- new net N$17: LED13.A, R13.1
- new net N$18: LED14.A, R14.1
- new net N$19: LED15.A, R15.1
- new net N$20: LED16.A, R16.1
- net N$1: no longer R10.2, R9.2
- net N$2: no longer LED10.C, LED9.C
Other:
- moved on the sheet: LED1, LED10, LED2, LED3, LED4, LED5, LED6, LED7, LED8, LED9, PAD1, PAD2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
