File: ring.brd (EAGLE design)
At the start: 82.5 x 87.6 mm, 22 parts

Commit message: placing
Parts:
- moved LED2 76.8 mm to (8.89, 68.6)
- moved LED5 65.7 mm to (14.0, 49.5)
- moved LED3 65.1 mm to (10.2, 62.2)
- moved LED1 63.7 mm to (7.62, 74.9)
- moved LED8 56.4 mm to (22.9, 34.3)
- moved R10 44.9 mm to (30.5, 25.4)
- moved LED4 38.4 mm to (11.4, 55.9)
- moved R2 29.3 mm to (7.62, 71.1)
- moved R9 22.2 mm to (24.1, 31.8)
- moved R6 16.5 mm to (15.2, 47.0)
- moved LED7 14.5 mm to (19.1, 39.4)
- moved LED9 14.5 mm to (27.9, 27.9)
- moved R8 13.1 mm to (21.6, 36.8)
- moved LED10 12.7 mm to (34.3, 22.9)
- moved LED6 12.0 mm to (16.5, 44.5)
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Changed lines of the file:
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@@
 </autorouter>
 <elements>
-<element name="LED1" library="led" package="KA-3528ASYC" value="" x="38.1" y="19.05"/>
-<element name="LED10" library="led" package="KA-3528ASYC" value="" x="44.45" y="15.24"/>
-<element name="LED2" library="led" package="KA-3528ASYC" value="" x="57.15" y="8.89"/>
-<element name="LED3" library="led" package="KA-3528ASYC" value="" x="50.8" y="11.43"/>
-<element name="LED4" library="led" package="KA-3528ASYC" value="" x="33.02" y="24.13"/>
-<element name="LED5" library="led" package="KA-3528ASYC" value="" x="63.5" y="6.35"/>
-<element name="LED6" library="led" package="KA-3528ASYC" value="" x="22.86" y="34.29"/>
-<element name="LED7" library="led" package="KA-3528ASYC" value="" x="27.94" y="27.94"/>
-<element name="LED8" library="led" package="KA-3528ASYC" value="" x="71.12" y="5.08"/>
-<element name="LED9" library="led" package="KA-3528ASYC" value="" x="19.05" y="39.37"/>
+<element name="LED1" library="led" package="KA-3528ASYC" value="" x="7.62" y="74.93"/>
+<element name="LED10" library="led" package="KA-3528ASYC" value="" x="34.29" y="22.86"/>
+<element name="LED2" library="led" package="KA-3528ASYC" value="" x="8.89" y="68.58"/>
+<element name="LED3" library="led" package="KA-3528ASYC" value="" x="10.16" y="62.23"/>
+<element name="LED4" library="led" package="KA-3528ASYC" value="" x="11.43" y="55.88"/>
+<element name="LED5" library="led" package="KA-3528ASYC" value="" x="13.97" y="49.53"/>
+<element name="LED6" library="led" package="KA-3528ASYC" value="" x="16.51" y="44.45"/>
+<element name="LED7" library="led" package="KA-3528ASYC" value="" x="19.05" y="39.37"/>
+<element name="LED8" library="led" package="KA-3528ASYC" value="" x="22.86" y="34.29"/>
+<element name="LED9" library="led" package="KA-3528ASYC" value="" x="27.94" y="27.94"/>
 <element name="PAD1" library="wirepad" package="SMD1,27-2,54" value="" x="83.82" y="3.81"/>
 <element name="PAD2" library="wirepad" package="SMD1,27-2,54" value="" x="86.36" y="3.81"/>
 <element name="R1" library="rcl" package="R0402" value="" x="7.62" y="77.47"/>
-<element name="R10" library="rcl" package="R0402" value="" x="8.89" y="64.77"/>
-<element name="R2" library="rcl" package="R0402" value="" x="16.51" y="43.18"/>
-<element name="R3" library="rcl" package="R0402" value="" x="11.43" y="53.34"/>
-<element name="R4" library="rcl" package="R0402" value="" x="10.16" y="55.88"/>
-<element name="R5" library="rcl" package="R0402" value="" x="10.16" y="59.69"/>
-<element name="R6" library="rcl" package="R0402" value="" x="8.89" y="62.23"/>
-<element name="R7" library="rcl" package="R0402" value="" x="16.51" y="45.72"/>
-<element name="R8" library="rcl" package="R0402" value="" x="15.24" y="48.26"/>
-<element name="R9" library="rcl" package="R0402" value="" x="12.7" y="50.8"/>
+<element name="R10" library="rcl" package="R0402" value="" x="30.48" y="25.4"/>
+<element name="R2" library="rcl" package="R0402" value="" x="7.62" y="71.12"/>
+<element name="R3" library="rcl" package="R0402" value="" x="8.89" y="64.77"/>
+<element name="R4" library="rcl" package="R0402" value="" x="10.16" y="59.69"/>
+<element name="R5" library="rcl" package="R0402" value="" x="12.7" y="53.34"/>
+<element name="R6" library="rcl" package="R0402" value="" x="15.24" y="46.99"/>
+<element name="R7" library="rcl" package="R0402" value="" x="17.78" y="41.91"/>
+<element name="R8" library="rcl" package="R0402" value="" x="21.59" y="36.83"/>
+<element name="R9" library="rcl" package="R0402" value="" x="24.13" y="31.75"/>
 </elements>
 <signals>
@@
 <contactref element="R9" pad="2"/>
 <contactref element="R10" pad="2"/>
-<wire x1="17.16" y1="43.18" x2="17.16" y2="45.72" width="0" layer="19" extent="1-1"/>
-<wire x1="15.89" y1="48.26" x2="17.16" y2="45.72" width="0" layer="19" extent="1-1"/>
-<wire x1="13.35" y1="50.8" x2="15.89" y2="48.26" width="0" layer="19" extent="1-1"/>
-<wire x1="12.08" y1="53.34" x2="17.16" y2="43.18" width="0" layer="19" extent="1-1"/>
-<wire x1="10.81" y1="55.88" x2="13.35" y2="50.8" width="0" layer="19" extent="1-1"/>
-<wire x1="10.81" y1="59.69" x2="10.81" y2="55.88" width="0" layer="19" extent="1-1"/>
-<wire x1="9.54" y1="62.23" x2="10.81" y2="59.69" width="0" layer="19" extent="1-1"/>
-<wire x1="9.54" y1="64.77" x2="9.54" y2="62.23" width="0" layer="19" extent="1-1"/>
-<wire x1="8.27" y1="77.47" x2="9.54" y2="64.77" width="0" layer="19" extent="1-1"/>
-<wire x1="83.82" y1="3.81" x2="17.16" y2="43.18" width="0" layer="19" extent="1-1"/>
+<wire x1="31.13" y1="25.4" x2="83.82" y2="3.81" width="0" layer="19" extent="1-1"/>
+<wire x1="24.78" y1="31.75" x2="31.13" y2="25.4" width="0" layer="19" extent="1-1"/>
+<wire x1="22.24" y1="36.83" x2="24.78" y2="31.75" width="0" layer="19" extent="1-1"/>
+<wire x1="18.43" y1="41.91" x2="22.24" y2="36.83" width="0" layer="19" extent="1-1"/>
+<wire x1="15.89" y1="46.99" x2="18.43" y2="41.91" width="0" layer="19" extent="1-1"/>
+<wire x1="13.35" y1="53.34" x2="15.89" y2="46.99" width="0" layer="19" extent="1-1"/>
+<wire x1="10.81" y1="59.69" x2="13.35" y2="53.34" width="0" layer="19" extent="1-1"/>
+<wire x1="9.54" y1="64.77" x2="10.81" y2="59.69" width="0" layer="19" extent="1-1"/>
+<wire x1="8.27" y1="71.12" x2="9.54" y2="64.77" width="0" layer="19" extent="1-1"/>
+<wire x1="8.27" y1="77.47" x2="8.27" y2="71.12" width="0" layer="19" extent="1-1"/>
 </signal>
 <signal name="N$2">
@@
 <contactref element="LED9" pad="C"/>
 <contactref element="LED10" pad="C"/>
-<wire x1="46" y1="15.24" x2="39.65" y2="19.05" width="0" layer="19" extent="1-1"/>
-<wire x1="86.36" y1="3.81" x2="46" y2="15.24" width="0" layer="19" extent="1-1"/>
-<wire x1="58.7" y1="8.89" x2="86.36" y2="3.81" width="0" layer="19" extent="1-1"/>
-<wire x1="65.05" y1="6.35" x2="58.7" y2="8.89" width="0" layer="19" extent="1-1"/>
-<wire x1="72.67" y1="5.08" x2="65.05" y2="6.35" width="0" layer="19" extent="1-1"/>
-<wire x1="52.35" y1="11.43" x2="86.36" y2="3.81" width="0" layer="19" extent="1-1"/>
-<wire x1="24.41" y1="34.29" x2="52.35" y2="11.43" width="0" layer="19" extent="1-1"/>
+<wire x1="35.84" y1="22.86" x2="86.36" y2="3.81" width="0" layer="19" extent="1-1"/>
+<wire x1="29.49" y1="27.94" x2="35.84" y2="22.86" width="0" layer="19" extent="1-1"/>
+<wire x1="24.41" y1="34.29" x2="29.49" y2="27.94" width="0" layer="19" extent="1-1"/>
 <wire x1="20.6" y1="39.37" x2="24.41" y2="34.29" width="0" layer="19" extent="1-1"/>
-<wire x1="34.57" y1="24.13" x2="52.35" y2="11.43" width="0" layer="19" extent="1-1"/>
-<wire x1="29.49" y1="27.94" x2="34.57" y2="24.13" width="0" layer="19" extent="1-1"/>
+<wire x1="18.06" y1="44.45" x2="20.6" y2="39.37" width="0" layer="19" extent="1-1"/>
+<wire x1="15.52" y1="49.53" x2="18.06" y2="44.45" width="0" layer="19" extent="1-1"/>
+<wire x1="12.98" y1="55.88" x2="15.52" y2="49.53" width="0" layer="19" extent="1-1"/>
+<wire x1="11.71" y1="62.23" x2="12.98" y2="55.88" width="0" layer="19" extent="1-1"/>
+<wire x1="10.44" y1="68.58" x2="11.71" y2="62.23" width="0" layer="19" extent="1-1"/>
+<wire x1="9.17" y1="74.93" x2="10.44" y2="68.58" width="0" layer="19" extent="1-1"/>
 </signal>
 <signal name="N$3">
 <contactref element="LED1" pad="A"/>
 <contactref element="R1" pad="1"/>
-<wire x1="6.97" y1="77.47" x2="36.55" y2="19.05" width="0" layer="19" extent="1-1"/>
+<wire x1="6.07" y1="74.93" x2="6.97" y2="77.47" width="0" layer="19" extent="1-1"/>
 </signal>
 <signal name="N$4">
 <contactref element="LED2" pad="A"/>
 <contactref element="R2" pad="1"/>
-<wire x1="15.86" y1="43.18" x2="55.6" y2="8.89" width="0" layer="19" extent="1-1"/>
+<wire x1="7.34" y1="68.58" x2="6.97" y2="71.12" width="0" layer="19" extent="1-1"/>
 </signal>
 <signal name="N$5">
 <contactref element="LED3" pad="A"/>
 <contactref element="R3" pad="1"/>
-<wire x1="10.78" y1="53.34" x2="49.25" y2="11.43" width="0" layer="19" extent="1-1"/>
+<wire x1="8.61" y1="62.23" x2="8.24" y2="64.77" width="0" layer="19" extent="1-1"/>
 </signal>
 <signal name="N$6">
 <contactref element="LED4" pad="A"/>
 <contactref element="R4" pad="1"/>
-<wire x1="9.51" y1="55.88" x2="31.47" y2="24.13" width="0" layer="19" extent="1-1"/>
+<wire x1="9.88" y1="55.88" x2="9.51" y2="59.69" width="0" layer="19" extent="1-1"/>
 </signal>
 <signal name="N$7">
 <contactref element="LED5" pad="A"/>
 <contactref element="R5" pad="1"/>
-<wire x1="9.51" y1="59.69" x2="61.95" y2="6.35" width="0" layer="19" extent="1-1"/>
+<wire x1="12.42" y1="49.53" x2="12.05" y2="53.34" width="0" layer="19" extent="1-1"/>
 </signal>
 <signal name="N$8">
 <contactref element="LED6" pad="A"/>
 <contactref element="R6" pad="1"/>
-<wire x1="8.24" y1="62.23" x2="21.31" y2="34.29" width="0" layer="19" extent="1-1"/>
+<wire x1="14.96" y1="44.45" x2="14.59" y2="46.99" width="0" layer="19" extent="1-1"/>
 </signal>
 <signal name="N$9">
 <contactref element="LED7" pad="A"/>
 <contactref element="R7" pad="1"/>
-<wire x1="15.86" y1="45.72" x2="26.39" y2="27.94" width="0" layer="19" extent="1-1"/>
+<wire x1="17.5" y1="39.37" x2="17.13" y2="41.91" width="0" layer="19" extent="1-1"/>
 </signal>
 <signal name="N$10">
 <contactref element="LED8" pad="A"/>
 <contactref element="R8" pad="1"/>
-<wire x1="69.57" y1="5.08" x2="14.59" y2="48.26" width="0" layer="19" extent="1-1"/>
+<wire x1="21.31" y1="34.29" x2="20.94" y2="36.83" width="0" layer="19" extent="1-1"/>
 </signal>
 <signal name="N$11">
 <contactref element="LED9" pad="A"/>
 <contactref element="R9" pad="1"/>
-<wire x1="12.05" y1="50.8" x2="17.5" y2="39.37" width="0" layer="19" extent="1-1"/>
+<wire x1="23.48" y1="31.75" x2="26.39" y2="27.94" width="0" layer="19" extent="1-1"/>
 </signal>
 <signal name="N$12">
 <contactref element="LED10" pad="A"/>
 <contactref element="R10" pad="1"/>
-<wire x1="8.24" y1="64.77" x2="42.9" y2="15.24" width="0" layer="19" extent="1-1"/>
+<wire x1="29.83" y1="25.4" x2="32.74" y2="22.86" width="0" layer="19" extent="1-1"/>
 </signal>
 </signals>

Commit message: dimensions
Parts:
- R1, R10, R2, R3, R4, R5, R6, R7, R8, R9: value (none) -> 330R
- moved R1 120.9 mm to (-11.4, -41.9)
- moved LED1 120.1 mm to (-5.08, -44.5)
- moved R2 112.5 mm to (-24.1, -36.8)
- moved LED2 112.4 mm to (-17.8, -40.6)
- moved LED3 103.8 mm to (-27.9, -34.3)
- moved R3 102.9 mm to (-33.0, -29.2)
- moved R4 93.7 mm to (-40.6, -19.1)
- moved LED4 93.4 mm to (-36.8, -24.1)
- moved LED5 84.6 mm to (-41.9, -14.0)
- moved R5 82.7 mm to (-43.2, -7.62)
- moved LED6 77.0 mm to (-44.5, -2.54)
- moved R6 72.9 mm to (-44.5, 5.08)
- moved LED7 68.7 mm to (-43.2, 10.2)
- moved R7 64.9 mm to (-41.9, 16.5)
- moved PAD1 64.8 mm to (26.7, 34.3)
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Other:
- board size 82.5 x 87.6 mm -> 82.6 x 96.8 mm

Commit message: skog
Parts:
- moved LED2 88.0 mm to (12.7, 41.9)
- moved R1 87.3 mm to (20.3, 39.4)
- moved PAD2 86.4 mm to (-3.81, -45.7)
- moved R2 85.9 mm to (3.81, 44.5)
- moved LED1 85.4 mm to (27.9, 34.3)
- moved R10 85.2 mm to (-11.4, -43.2)
- moved PAD1 84.7 mm to (-1.27, -45.7)
- moved LED3 82.0 mm to (-5.08, 44.5)
- moved LED10 78.8 mm to (-17.8, -40.6)
- moved R3 75.5 mm to (-11.4, 43.2)
- moved R9 71.1 mm to (-26.7, -35.6)
- moved LED4 65.6 mm to (-20.3, 39.4)
- moved LED9 62.3 mm to (-33.0, -30.5)
- moved R4 56.4 mm to (-26.7, 35.6)
- moved R8 49.6 mm to (-38.1, -22.9)
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Other:
- board size 82.6 x 96.8 mm -> 90 x 90 mm

Commit message: angled
Parts:
- moved R2 21.8 mm to (22.9, 33.9), turned to 160 degrees
- moved R3 19.7 mm to (8.05, 40.2), turned to 180 degrees
- moved R1 19.6 mm to (32.7, 24.2), turned to 136 degrees
- moved R4 17.5 mm to (-9.71, 39.8), turned to 204 degrees
- moved R5 15.7 mm to (-25.4, 32.1), turned to 228 degrees
- moved LED3 15.6 mm to (6.72, 34.3), turned to 170 degrees
- moved LED2 14.4 mm to (19.4, 29.2), turned to 148 degrees
- moved LED4 13.2 mm to (-8.25, 33.9), turned to 194 degrees
- moved LED1 13.1 mm to (27.8, 21.2), turned to 126 degrees
- moved R6 11.6 mm to (-36.7, 18.5), turned to 252 degrees
- moved R10 11.0 mm to (-20.1, -36.3), turned to 342 degrees
- moved R9 10.7 mm to (-32.0, -26.3), turned to 322 degrees
- moved R7 10.6 mm to (-40.8, 3.64), turned to 276 degrees
- moved R8 10.5 mm to (-39.3, -12.4), turned to 300 degrees
- moved LED5 10.5 mm to (-21.7, 27.5), turned to 218 degrees
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Other:
- outline, holes or cut-outs redrawn

Commit message: fin
Parts:
- R1, R10, R2, R3, R4, R5, R6, R7, R8, R9: device rcl:R0402 -> rcl:R0805W
- moved R1 1.92 mm to (34.0, 25.6), turned to 36 degrees
- moved R2 1.68 mm to (23.5, 35.4), turned to 58 degrees
- moved R3 1.52 mm to (7.93, 41.7), turned to 80 degrees
- moved R5 1.48 mm to (-26.2, 33.4), turned to 128 degrees
- moved R4 1.45 mm to (-10.1, 41.2), turned to 104 degrees
- moved R7 1.39 mm to (-42.2, 3.81), turned to 174 degrees
- moved R6 1.39 mm to (-37.8, 19.4), turned to 150 degrees
- moved R8 1.39 mm to (-40.6, -12.3), turned to 198 degrees
- moved LED7 1.19 mm to (-35.8, 3.23)
- moved LED6 1.18 mm to (-32.0, 16.4)
- moved LED8 1.15 mm to (-34.4, -10.4)
- moved LED3 1.08 mm to (6.91, 35.3)
- moved R9 1.07 mm to (-33.0, -26.6), turned to 220 degrees
- moved LED1 1.07 mm to (28.7, 21.7)
- moved LED2 1.07 mm to (19.9, 30.1)
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Routing:
- net N$2: track 0.00 -> 294.6 mm
- net N$1: track 0.00 -> 173.9 mm
- net N$9: track 0.00 -> 7.07 mm
- net N$10: track 0.00 -> 7.04 mm
- net N$8: track 0.00 -> 7.04 mm
- net N$12: track 0.00 -> 7.03 mm
- net N$5: track 0.00 -> 7.00 mm
- net N$3: track 0.00 -> 6.98 mm
- net N$4: track 0.00 -> 6.95 mm
- net N$7: track 0.00 -> 6.87 mm
- net N$6: track 0.00 -> 6.86 mm
- net N$11: track 0.00 -> 6.74 mm
Other:
- board size 90 x 90 mm -> 83.1 x 90 mm

Commit message: curve
Routing:
- net N$2: track 294.6 -> 291.9 mm
Other:
- outline, holes or cut-outs redrawn

Commit message: new
Parts:
- added LED11, LED12, LED13, LED14, LED15, LED16: (no value), led:KA-3528ASYC
- added PAD3, PAD4: (no value), wirepad:SMD1,27-2,54
- added R11, R12, R13, R14, R15, R16: 330R, rcl:R0805W
- moved LED3 200.3 mm to (-90.0, -140.0), turned to 0 degrees
- moved LED1 189.6 mm to (-85.0, -130.0), turned to 0 degrees
- moved LED4 189.0 mm to (-80.0, -140.0), turned to 0 degrees
- moved LED2 186.1 mm to (-75.0, -130.0), turned to 0 degrees
- moved R1 176.5 mm to (-90.0, -100.0), turned to 0 degrees
- moved LED5 174.8 mm to (-70.0, -140.0), turned to 0 degrees
- moved LED6 171.5 mm to (-90.0, -145.0), turned to 0 degrees
- moved R4 171.0 mm to (-90.0, -110.0), turned to 0 degrees
- moved R2 170.4 mm to (-80.0, -100.0), turned to 0 degrees
- moved R3 161.7 mm to (-70.0, -100.0), turned to 0 degrees
- moved LED7 154.7 mm to (-80.0, -145.0), turned to 0 degrees
- moved R5 153.1 mm to (-80.0, -110.0), turned to 0 degrees
- moved LED8 139.2 mm to (-70.0, -145.0), turned to 0 degrees
- moved R6 133.3 mm to (-70.0, -110.0), turned to 0 degrees
- moved R7 132.7 mm to (-90.0, -120.0), turned to 0 degrees
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Connections:
- new net N$11: PAD3.1, R10.2, R11.2, R12.2, R13.2, R14.2, R15.2, R16.2, R9.2
- new net N$12: LED10.C, LED11.C, LED12.C, LED13.C, LED14.C, LED15.C, LED16.C, LED9.C, PAD4.1
- new net N$15: LED11.A, R11.1
- new net N$16: LED12.A, R12.1
- new net N$17: LED13.A, R13.1
- new net N$18: LED14.A, R14.1
- new net N$19: LED15.A, R15.1
- new net N$20: LED16.A, R16.1
- net N$1: no longer R10.2, R9.2
- net N$2: no longer LED10.C, LED9.C
Routing:
- net N$2: track 291.9 -> 0.00 mm
- net N$1: track 173.8 -> 0.00 mm
- net N$9: track 7.07 -> 0.00 mm
- net N$10: track 7.04 -> 0.00 mm
- net N$8: track 7.04 -> 0.00 mm
- net N$14: track 7.03 -> 0.00 mm
- net N$5: track 7.00 -> 0.00 mm
- net N$3: track 6.98 -> 0.00 mm
- net N$4: track 6.95 -> 0.00 mm
- net N$7: track 6.87 -> 0.00 mm
- net N$6: track 6.86 -> 0.00 mm
- net N$13: track 6.74 -> 0.00 mm
Other:
- board size 83.1 x 90 mm -> 174.9 x 190 mm

Commit message: placing
Parts:
- moved LED8 261.6 mm to (45.0, 90.0)
- moved R8 241.9 mm to (40.0, 90.0)
- moved LED7 241.7 mm to (20.0, 75.0)
- moved R7 221.5 mm to (15.0, 75.0)
- moved LED6 219.3 mm to (0.00, 55.0)
- moved LED5 180.3 mm to (-10.0, 30.0)
- moved R6 177.3 mm to (-5.00, 55.0)
- moved PAD2 171.0 mm to (75.0, -85.0)
- moved LED4 156.5 mm to (-10.0, 0.00)
- moved R5 154.4 mm to (-15.0, 30.0)
- moved PAD1 154.0 mm to (80.0, -85.0)
- moved LED3 139.0 mm to (-5.00, -30.0)
- moved LED1 134.6 mm to (40.0, -80.0)
- moved R4 133.1 mm to (-15.0, 0.00)
- moved R1 126.6 mm to (35.0, -80.0)
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